File: kicad/bobbycar-emergency-hardware.kicad_sch (KiCad schematic)
At the start: 43 parts, among them J1 CAN2, J2 PROG, Q1 SS8050_C2150, Q2 SS8050_C2150, SW1 ANALOG_LEFT, U1 SN65HVD231, U2 ESP32-WROOM-32, U3 AMS1117-3.3, U4 MPM2359, U5 CH343G

Commit message: PCB Files and more screenshots
Parts:
- U2: LCSC Part # C701343 -> C701342
Changed lines of the file:
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@@
       (effects (font (size 1.27 1.27)) hide)
     )
-    (property "LCSC Part #" "C701343" (id 4) (at 63.5 69.85 0)
+    (property "LCSC Part #" "C701342" (id 4) (at 63.5 69.85 0)
       (effects (font (size 1.27 1.27)) hide)
     )

Commit message: Fixed JLCPCB, added marks for orientation etc
Parts:
- C13, C8: LCSC Part # C45783 -> C32375
Changed lines of the file:
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@@
       (effects (font (size 1.27 1.27)) hide)
     )
-    (property "LCSC Part #" "C45783" (id 4) (at 220.98 59.69 0)
+    (property "LCSC Part #" "C32375" (id 4) (at 220.98 59.69 0)
       (effects (font (size 1.27 1.27)) hide)
     )
@@
       (effects (font (size 1.27 1.27)) hide)
     )
-    (property "LCSC Part #" "C45783" (id 4) (at 152.4 54.61 0)
-      (effects (font (size 1.27 1.27)) hide)
-    )
+    (property "LCSC Part #" "C32375" (id 4) (at 152.4 54.61 0)
+      (effects (font (size 1.27 1.27)) hide)
+    )
